File: XboxSerialAdapter.brd (EAGLE design)
At the start: 42.6 x 43.9 mm, 21 parts, among them IC1 CP2102, J2 0475900001, U1 LPC47M192

Commit message: Update: crystal
Parts:
- Q1: device crystal-geyer_V1_0:5.0X3.2_KXO-V99 -> xbox:SCTF_C387229
- moved Q1 0.91 mm to (5.98, 70.4)
Connections:
- new net GND/NC: Q1.1
Changed lines of the file:
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@@
 <attribute name="VALUE" x="8.255" y="41.91" size="1.27" layer="27" rot="R90" align="top-center"/>
-</element>
-<element name="Q1" library="crystal-geyer_V1_0" library_urn="urn:adsk.eagle:library:203" package="5.0X3.2_KXO-V99" package3d_urn="urn:adsk.eagle:package:11948/1" value="" x="5.08" y="70.485" smashed="yes">
-<attribute name="LCSC_PART" value="C387229" x="5.08" y="70.485" size="1.778" layer="27" display="off"/>
-<attribute name="NAME" x="2.44" y="72.385" size="1.016" layer="25"/>
-<attribute name="VALUE" x="2.44" y="67.585" size="1.016" layer="27"/>
 </element>
 <element name="R5" library="SparkFun" package="0603-RES" value="680" x="19.05" y="66.04" smashed="yes">
@@
 <attribute name="POPULARITY" value="26" x="24.39035" y="75.3745" size="1.778" layer="27" rot="R270" display="off"/>
 <attribute name="VALUE" x="19.11985" y="68.5927" size="1.27" layer="27"/>
+</element>
+<element name="Q1" library="xbox" package="SCTF_C387229" package3d_urn="urn:adsk.eagle:package:11966/1" value="" x="5.9817" y="70.35165" smashed="yes">
+<attribute name="LCSC_PART" value="C387229" x="5.9817" y="70.35165" size="1.778" layer="27" display="off"/>
+<attribute name="NAME" x="3.2317" y="72.45165" size="1.016" layer="25"/>
+<attribute name="VALUE" x="3.2317" y="67.25165" size="1.016" layer="27"/>
 </element>
 </elements>
@@
 <contactref element="C3" pad="2"/>
 <contactref element="C2" pad="2"/>
-<contactref element="Q1" pad="2"/>
 <contactref element="C4" pad="2"/>
 <contactref element="C5" pad="2"/>
@@
 <wire x1="25.146" y1="70.104" x2="25.2025" y2="70.0475" width="0.1524" layer="1"/>
 <wire x1="25.146" y1="70.104" x2="25.146" y2="70.08005" width="0.1524" layer="1"/>
+<contactref element="Q1" pad="2"/>
 <wire x1="8.285" y1="75.43" x2="9.21" y2="75.105" width="0" layer="19" extent="1-1"/>
 <wire x1="19.9" y1="63.5" x2="25.06" y2="62.37" width="0" layer="19" extent="1-1"/>
@@
 <wire x1="25.7556" y1="67.9704" x2="25.06" y2="62.37" width="0" layer="19" extent="1-1"/>
 <wire x1="25.2984" y1="68.4276" x2="25.7556" y2="67.9704" width="0" layer="19" extent="1-1"/>
+<wire x1="7.2517" y1="69.20165" x2="6.77" y2="63.5" width="0" layer="19" extent="1-1"/>
 <wire x1="16.96015" y1="76.8985" x2="11.16" y2="78.105" width="0" layer="19" extent="1-1"/>
 <wire x1="37.81" y1="44.62" x2="37.81" y2="56.62" width="0" layer="19" extent="1-1"/>
@@
 <contactref element="U1" pad="53"/>
 <contactref element="C5" pad="1"/>
-<contactref element="Q1" pad="4"/>
 <contactref element="C2" pad="1"/>
 <contactref element="R1" pad="2"/>
@@
 <wire x1="14.478" y1="63.5508" x2="14.39" y2="63.5" width="0.1524" layer="1"/>
 <wire x1="4.572" y1="65.9892" x2="4.66" y2="66.04" width="0.1524" layer="1"/>
-<wire x1="3.81" y1="71.628" x2="3.83" y2="71.635" width="0.1524" layer="1"/>
 <wire x1="8.47" y1="63.40105" x2="8.47" y2="63.5" width="0.1524" layer="1"/>
 <wire x1="16.764" y1="49.2252" x2="19.812" y2="46.1772" width="0.1524" layer="1"/>
@@
 <wire x1="14.3256" y1="63.5508" x2="14.39" y2="63.5" width="0.1524" layer="1"/>
 <wire x1="8.5344" y1="63.5508" x2="8.47" y2="63.5" width="0.1524" layer="1"/>
-<wire x1="3.9624" y1="71.0184" x2="3.9624" y2="71.628" width="0.1524" layer="1"/>
-<wire x1="4.8768" y1="70.104" x2="3.9624" y2="71.0184" width="0.1524" layer="1"/>
 <wire x1="4.8768" y1="66.294" x2="4.8768" y2="66.9036" width="0.1524" layer="1"/>
-<wire x1="4.8768" y1="66.9036" x2="4.8768" y2="70.104" width="0.1524" layer="1"/>
 <wire x1="4.7244" y1="66.1416" x2="4.8768" y2="66.294" width="0.1524" layer="1"/>
-<wire x1="3.9624" y1="71.628" x2="3.83" y2="71.635" width="0.1524" layer="1"/>
 <wire x1="4.7244" y1="66.1416" x2="4.66" y2="66.04" width="0.1524" layer="1"/>
 <wire x1="28.194" y1="63.5508" x2="28.4988" y2="63.246" width="0.1524" layer="1"/>
@@
 <wire x1="1.8288" y1="66.294" x2="1.8288" y2="59.8932" width="0.1524" layer="1"/>
 <wire x1="2.4384" y1="66.9036" x2="1.8288" y2="66.294" width="0.1524" layer="1"/>
-<wire x1="4.8768" y1="66.9036" x2="2.4384" y2="66.9036" width="0.1524" layer="1"/>
+<wire x1="4.8768" y1="66.9036" x2="3.5052" y2="66.9036" width="0.1524" layer="1"/>
+<wire x1="3.5052" y1="66.9036" x2="2.4384" y2="66.9036" width="0.1524" layer="1"/>
 <wire x1="14.3256" y1="52.1208" x2="15.24" y2="52.1208" width="0.1524" layer="1"/>
 <wire x1="13.2588" y1="53.1876" x2="14.3256" y2="52.1208" width="0.1524" layer="1"/>
@@
 <wire x1="2.5908" y1="53.4924" x2="7.0104" y2="53.4924" width="0.1524" layer="1"/>
 <wire x1="15.24" y1="52.1208" x2="15.24" y2="52.07" width="0.1524" layer="1"/>
+<contactref element="Q1" pad="4"/>
+<wire x1="4.572" y1="71.0184" x2="4.572" y2="71.4756" width="0.1524" layer="1"/>
+<wire x1="3.5052" y1="69.9516" x2="4.572" y2="71.0184" width="0.1524" layer="1"/>
+<wire x1="3.5052" y1="66.9036" x2="3.5052" y2="69.9516" width="0.1524" layer="1"/>
+<wire x1="4.572" y1="71.4756" x2="4.7117" y2="71.50165" width="0.1524" layer="1"/>
 </signal>
 <signal name="N$1">
@@
 </signal>
 <signal name="CLOCK">
-<contactref element="Q1" pad="3"/>
 <contactref element="J1" pad="3"/>
 <contactref element="U1" pad="19"/>
-<wire x1="6.2484" y1="72.0852" x2="6.2484" y2="71.7804" width="0.1524" layer="1"/>
-<wire x1="6.2484" y1="71.7804" x2="6.33" y2="71.635" width="0.1524" layer="1"/>
 <wire x1="38.7096" y1="50.5968" x2="37.9476" y2="50.5968" width="0.1524" layer="1"/>
 <wire x1="37.9476" y1="50.5968" x2="37.81" y2="50.62" width="0.1524" layer="1"/>
-<wire x1="3.9624" y1="74.3712" x2="6.2484" y2="72.0852" width="0.1524" layer="1"/>
 <wire x1="3.9624" y1="77.8764" x2="3.9624" y2="74.3712" width="0.1524" layer="1"/>
 <wire x1="5.4864" y1="79.4004" x2="3.9624" y2="77.8764" width="0.1524" layer="1"/>
@@
 <wire x1="39.624" y1="72.6948" x2="39.624" y2="76.8096" width="0.1524" layer="1"/>
 <wire x1="38.1" y1="71.1708" x2="39.624" y2="72.6948" width="0.1524" layer="1"/>
-<wire x1="6.2484" y1="72.0852" x2="6.33" y2="71.635" width="0.1524" layer="1"/>
 <wire x1="38.1" y1="71.1708" x2="38.1" y2="71.12" width="0.1524" layer="1"/>
 <wire x1="39.1668" y1="51.054" x2="38.7096" y2="50.5968" width="0.1524" layer="1"/>
@@
 <wire x1="38.7096" y1="50.5968" x2="37.81" y2="50.62" width="0.1524" layer="1"/>
 <via x="39.1668" y="51.054" extent="1-16" drill="0.254"/>
+<contactref element="Q1" pad="3"/>
+<wire x1="6.7056" y1="71.628" x2="7.1628" y2="71.628" width="0.1524" layer="1"/>
+<wire x1="3.9624" y1="74.3712" x2="6.7056" y2="71.628" width="0.1524" layer="1"/>
+<wire x1="7.1628" y1="71.628" x2="7.2517" y2="71.50165" width="0.1524" layer="1"/>
+</signal>
+<signal name="GND/NC">
+<contactref element="Q1" pad="1"/>
 </signal>
 </signals>

Commit message: Update: files
Routing:
- net GND: track 6.75 -> 8.47 mm, vias 2 -> 15
- net VCC: track 126.7 -> 125.8 mm
- net LAD0: track 41.5 -> 40.8 mm
- net D-: track 23.6 -> 22.9 mm
- net N$6: track 43.2 -> 42.6 mm
