File: XboxSerialAdapter.sch (EAGLE design)
At the start: 21 parts, among them IC1 CP2102, J2 0475900001, U1 LPC47M192

Commit message: Update: crystal
Parts:
- Q1: device crystal-geyer_V1_0:KXO-PXO/XO-V99 -> xbox:SCTF_C3872291
Connections:
- net VCC: now also Q1.VCC; no longer Q1.VDD
Changed lines of the file:
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@@
 <attribute name="LCSC_PART" value="C191538"/>
-</part>
-<part name="Q1" library="crystal-geyer_V1_0" library_urn="urn:adsk.eagle:library:203" deviceset="KXO-PXO/XO-V" device="99" package3d_urn="urn:adsk.eagle:package:11948/1">
-<attribute name="LCSC_PART" value="C387229"/>
 </part>
 <part name="P+2" library="supply1" library_urn="urn:adsk.eagle:library:371" deviceset="VCC" device=""/>
@@
 <part name="TX" library="led" library_urn="urn:adsk.eagle:library:259" deviceset="LED" device="CHIP-LED0603" package3d_urn="urn:adsk.eagle:package:15819/3" value="Green">
 <attribute name="LCSC_PART" value="C125113"/>
+</part>
+<part name="Q1" library="xbox" deviceset="SCTF_C387229" device="1" package3d_urn="urn:adsk.eagle:package:11966/1">
+<attribute name="LCSC_PART" value="C387229"/>
 </part>
 </parts>
@@
 <attribute name="LCSC_PART" x="30.48" y="134.62" size="1.778" layer="96"/>
 </instance>
-<instance part="Q1" gate="G$1" x="68.58" y="78.74" smashed="yes">
-<attribute name="NAME" x="60.96" y="86.995" size="1.778" layer="95"/>
-<attribute name="VALUE" x="60.96" y="68.58" size="1.778" layer="96"/>
-<attribute name="LCSC_PART" x="68.58" y="78.74" size="1.778" layer="96"/>
-</instance>
 <instance part="P+2" gate="VCC" x="45.72" y="91.44" smashed="yes">
 <attribute name="VALUE" x="43.18" y="92.71" size="1.778" layer="96"/>
@@
 <attribute name="VALUE" x="183.515" y="140.208" size="1.778" layer="96" rot="R90"/>
 <attribute name="LCSC_PART" x="180.34" y="144.78" size="1.778" layer="96"/>
+</instance>
+<instance part="Q1" gate="G$1" x="68.58" y="78.74" smashed="yes">
+<attribute name="NAME" x="60.96" y="86.995" size="1.778" layer="95"/>
+<attribute name="LCSC_PART" x="68.58" y="78.74" size="1.778" layer="96"/>
 </instance>
 </instances>
@@
 <wire x1="30.48" y1="83.82" x2="22.86" y2="83.82" width="0.1524" layer="91"/>
 <wire x1="22.86" y1="83.82" x2="22.86" y2="73.66" width="0.1524" layer="91"/>
-<pinref part="Q1" gate="G$1" pin="GND"/>
 <wire x1="22.86" y1="73.66" x2="58.42" y2="73.66" width="0.1524" layer="91"/>
 <wire x1="22.86" y1="83.82" x2="12.7" y2="83.82" width="0.1524" layer="91"/>
 <junction x="22.86" y="83.82"/>
 <pinref part="GND3" gate="1" pin="GND"/>
+<pinref part="Q1" gate="G$1" pin="GND"/>
 </segment>
 <segment>
@@
 </segment>
 <segment>
-<pinref part="Q1" gate="G$1" pin="VDD"/>
 <wire x1="58.42" y1="83.82" x2="45.72" y2="83.82" width="0.1524" layer="91"/>
 <pinref part="P+2" gate="VCC" pin="VCC"/>
@@
 <junction x="45.72" y="83.82"/>
 <pinref part="C2" gate="G$1" pin="1"/>
+<pinref part="Q1" gate="G$1" pin="VCC"/>
 </segment>
 <segment>
@@
 <net name="CLOCK" class="0">
 <segment>
-<pinref part="Q1" gate="G$1" pin="OUT"/>
 <wire x1="78.74" y1="78.74" x2="93.98" y2="78.74" width="0.1524" layer="91"/>
 <label x="86.36" y="78.74" size="1.778" layer="95"/>
-</segment>
-<segment>
+<pinref part="Q1" gate="G$1" pin="OUT"/>
+</segment>
+<segment>
